File: Tools/eda/templates/6U_Eurocard/6U_Eurocard.kicad_pcb (KiCad board)
At the start: 2 copper layers, 233.3 x 160 mm, 2 parts, among them J2 DIN41612_03x32_C_Split

Commit message: Cleans up bus allocations across cards
Parts:
- added REF**: MountingHole_2.5mm, MountingHole:MountingHole_2.5mm, F.Cu at (93.6, 70.4)
- added REF**: MountingHole_2.5mm, MountingHole:MountingHole_2.5mm, F.Cu at (316.9, 70.4)
- moved J2 110.1 mm to (308.7, 220.1)
- moved J1 110.1 mm to (179.2, 220.1)
- renumbered REF** to J1
Other:
- board size 233.3 x 160 mm -> 233.4 x 160 mm
